File: 1602-backpack.kicad_sch (KiCad schematic)
At the start: 7 parts, among them J1 Display, J2 Full, J3 Minimal

Commit message: Finalise layout and round corners
Parts:
- removed J1: Display, Connector_PinSocket_2.54mm:PinSocket_1x16_P2.54mm_Vertical, symbol Connector:Conn_01x16_Female
- added DS1: WC1602A, Connector_PinSocket_2.54mm:PinSocket_1x16_P2.54mm_Vertical, symbol Display_Character:WC1602A
Connections:
- net A: now also DS1.15 (LED(+))
- net D0: now also DS1.7 (D0)
- net D1: now also DS1.8 (D1)
- net D2: now also DS1.9 (D2)
- net D3: now also DS1.10 (D3)
- net D4: now also DS1.11 (D4)
- net D5: now also DS1.12 (D5)
- net D6: now also DS1.13 (D6)
- net D7: now also DS1.14 (D7)
- net E: now also DS1.6 (E)
- net K: now also DS1.16 (LED(-))
- net RS: now also DS1.4 (RS)
- net RW: now also JP1.1 (A), DS1.5 (R/W); no longer JP1.2 (B)
- net VDD: now also DS1.2 (VDD)
- net VSS: now also JP1.2 (B), DS1.1 (VSS); no longer JP1.1 (A)
- net VE renamed V0
- net V0: now also DS1.3 (VO)
Other:
- moved on the sheet: J2, J3, JP1, JP2, JP3, RV1
